Commit message: New try

File: psa_robot_description/urdf/astra.urdf.xacro (robot description, xacro)
@@ -17,5 +17,5 @@
         <origin xyz="-0.03 -0.06 0" rpy="${pi} 0 ${pi/2}"/>
         <geometry>
-          <mesh filename="package://softbot_description/meshes/astra2/astra2.dae" scale="1 1 1"/>
+          <mesh filename="package://psa_robot_description/meshes/astra2/astra2.dae" scale="1 1 1"/>
         </geometry>
       </visual>

File: psa_robot_description/urdf/psa_robot.gazebo.macro.xacro (robot description, xacro)
@@ -70,5 +70,5 @@
   </gazebo>
   <!--Using gazebo or ROS native controller for differential drives.-->
-  <xacro:include filename="$(find softbot_description)/urdf/ros_diff_drive.gazebo.xacro"/>
+  <xacro:include filename="$(find psa_robot_description)/urdf/ros_diff_drive.gazebo.xacro"/>
   <gazebo>
     <plugin name="imu_plugin" filename="libgazebo_ros_imu.so">

File: psa_robot_description/urdf/psa_robot.urdf.xacro (robot description, xacro)
@@ -1,4 +1,4 @@
 <?xml version="1.0" ?>
-<robot name="softbot" xmlns:xacro="http://ros.org/wiki/xacro">
+<robot name="psa_robot" xmlns:xacro="http://ros.org/wiki/xacro">
   <!--  Xacro description of turtlebot robot waffle pi used to play team hunt.-->
   <!--  Miguel Riem Oliveira-->
